Commit message: Add collision for MH50 II 20

File: motoman_mh50_support/urdf/mh50ii20_macro.xacro (robot description, xacro)
@@ -42,6 +42,7 @@
             </visual>
             <collision>
+                <origin xyz="-0.145 0 -0.540" rpy="0 0 0" />
                 <geometry>
-                    <mesh filename="package://motoman_mh50_support/meshes/collision/mh50_link_2_l.stl"/>
+                    <mesh filename="package://motoman_mh50_support/meshes/collision/mh50ii20_link_2_l.stl"/>
                 </geometry>
             </collision>
@@ -56,6 +57,7 @@
             </visual>
             <collision>
+                <origin xyz="-0.145 0 -1.690" rpy="0 0 0" />
                 <geometry>
-                    <mesh filename="package://motoman_mh50_support/meshes/collision/mh50_link_3_u.stl"/>
+                    <mesh filename="package://motoman_mh50_support/meshes/collision/mh50ii20_link_3_u.stl"/>
                 </geometry>
             </collision>
@@ -70,6 +72,7 @@
             </visual>
             <collision>
+                <origin xyz="-1.945 0 -1.890" rpy="0 0 0" />
                 <geometry>
-                    <mesh filename="package://motoman_mh50_support/meshes/collision/mh50_link_4_r.stl"/>
+                    <mesh filename="package://motoman_mh50_support/meshes/collision/mh50ii20_link_4_r.stl"/>
                 </geometry>
             </collision>
@@ -84,6 +87,7 @@
             </visual>
             <collision>
+                <origin xyz="-1.945 0 -1.890" rpy="0 0 0" />
                 <geometry>
-                    <mesh filename="package://motoman_mh50_support/meshes/collision/mh50_link_5_b.stl"/>
+                    <mesh filename="package://motoman_mh50_support/meshes/collision/mh50ii20_link_5_b.stl"/>
                 </geometry>
             </collision>
@@ -98,6 +102,7 @@
             </visual>
             <collision>
+                <origin xyz="-1.945 0 -1.890" rpy="0 0 0" />
                 <geometry>
-                    <mesh filename="package://motoman_mh50_support/meshes/collision/mh50_link_6_t.stl"/>
+                    <mesh filename="package://motoman_mh50_support/meshes/collision/mh50ii20_link_6_t.stl"/>
                 </geometry>
             </collision>

Commit message: Move yaskawa_blue material out of macro for multirobot

File: motoman_mh50_support/urdf/mh50ii20_macro.xacro (robot description, xacro)
@@ -1,9 +1,9 @@
 <?xml version="1.0" ?>
 <robot xmlns:xacro="http://ros.org/wiki/xacro">
+    <!-- Properties -->
+    <material name="yaskawa_blue">
+        <color rgba="0.12941 0.14902 0.74902 1" />
+    </material>
     <xacro:macro name="motoman_mh50ii20" params="prefix">
-        <!-- Properties -->
-        <material name="yaskawa_blue">
-            <color rgba="0.12941 0.14902 0.74902 1" />
-        </material>
         <!-- link list -->
         <link name="${prefix}base_link">

Commit message: Set joint limits to something reasonable

File: motoman_mh50_support/urdf/mh50ii20_macro.xacro (robot description, xacro)
@@ -123,5 +123,5 @@
             <origin xyz="0.145 0 0" rpy="0 0 0" />
             <axis xyz="0 1 0" />
-            <limit lower="-1.57079" upper="2.35619" effort="6276.26" velocity="3.103"/>
+            <limit lower="${radians(-90)}" upper="${radians(135)}" effort="6276.26" velocity="${radians(178)}"/>
         </joint>
         <joint name="${prefix}joint_3_u" type="revolute">
@@ -130,5 +130,5 @@
             <origin xyz="0 0 1.150" rpy="0 0 0" />
             <axis xyz="0 -1 0" />
-            <limit lower="-1.39626" upper="3.59538" effort="2745.86" velocity="3.106"/>
+            <limit lower="${radians(-70)}" upper="${radians(70)}" effort="2745.86" velocity="${radians(178)}"/>
         </joint>
         <joint name="${prefix}joint_4_r" type="revolute">
@@ -137,5 +137,5 @@
             <origin xyz="1.800 0 0.200" rpy="0 0 0"/>
             <axis xyz="-1 0 0" />
-            <limit lower="-6.28319" upper="6.28319" effort="823.76" velocity="4.363"/>
+            <limit lower="${radians(-190)}" upper="${radians(190)}" effort="823.76" velocity="${radians(400)}"/>
         </joint>
         <joint name="${prefix}joint_5_b" type="revolute">
@@ -144,5 +144,5 @@
             <origin xyz="0 0 0" rpy="0 0 0" />
             <axis xyz="0 -1 0" />
-            <limit lower="-2.18167" upper="2.18167" effort="706.08" velocity="4.363"/>
+            <limit lower="${radians(-140)}" upper="${radians(140)}" effort="706.08" velocity="${radians(400)}"/>
         </joint>
         <joint name="${prefix}joint_6_t" type="revolute">
@@ -151,5 +151,5 @@
             <origin xyz="0 0 0" rpy="0 0 0" />
             <axis xyz="-1 0 0" />
-            <limit lower="-6.2831" upper="6.2831" effort="333.43" velocity="6.283"/>
+            <limit lower="-6.2831" upper="6.2831" effort="333.43" velocity="${radians(600)}"/>
         </joint>
         <joint name="${prefix}joint_6_t-tool0" type="fixed">

Commit message: Use motoman_resources for mh50-ii-20
I would need to go back and disable auto formatting to apply this to existing robots without changing every single line.

File: motoman_mh50_support/urdf/mh50ii20_macro.xacro (robot description, xacro)
@@ -1,8 +1,5 @@
 <?xml version="1.0" ?>
 <robot xmlns:xacro="http://ros.org/wiki/xacro">
-    <!-- Properties -->
-    <material name="yaskawa_blue">
-        <color rgba="0.12941 0.14902 0.74902 1" />
-    </material>
+    <xacro:include filename="$(find motoman_resources)/urdf/common_materials.xacro"/>
     <xacro:macro name="motoman_mh50ii20" params="prefix">
         <!-- link list -->
@@ -12,5 +9,5 @@
                     <mesh filename="package://motoman_mh50_support/meshes/visual/mh50_base_link.stl"/>
                 </geometry>
-                <material name="yaskawa_blue"/>
+                <xacro:material_yaskawa_blue />
             </visual>
             <collision>
@@ -25,5 +22,5 @@
                     <mesh filename="package://motoman_mh50_support/meshes/visual/mh50_link_1_s.stl"/>
                 </geometry>
-                <material name="yaskawa_blue"/>
+                <xacro:material_yaskawa_blue />
             </visual>
             <collision>
@@ -39,5 +36,5 @@
                     <mesh filename="package://motoman_mh50_support/meshes/visual/mh50ii20_link_2_l.stl"/>
                 </geometry>
-                <material name="yaskawa_blue"/>
+                <xacro:material_yaskawa_blue />
             </visual>
             <collision>
@@ -54,5 +51,5 @@
                     <mesh filename="package://motoman_mh50_support/meshes/visual/mh50ii20_link_3_u.stl"/>
                 </geometry>
-                <material name="yaskawa_blue"/>
+                <xacro:material_yaskawa_blue />
             </visual>
             <collision>
@@ -69,5 +66,5 @@
                     <mesh filename="package://motoman_mh50_support/meshes/visual/mh50ii20_link_4_r.stl"/>
                 </geometry>
-                <material name="yaskawa_blue"/>
+                <xacro:material_yaskawa_blue />
             </visual>
             <collision>
@@ -84,5 +81,5 @@
                     <mesh filename="package://motoman_mh50_support/meshes/visual/mh50ii20_link_5_b.stl"/>
                 </geometry>
-                <material name="yaskawa_blue"/>
+                <xacro:material_yaskawa_blue />
             </visual>
             <collision>
@@ -99,5 +96,5 @@
                     <mesh filename="package://motoman_mh50_support/meshes/visual/mh50ii20_link_6_t.stl"/>
                 </geometry>
-                <material name="yaskawa_blue"/>
+                <xacro:material_yaskawa_blue />
             </visual>
             <collision>
